Commit message: Backup: 重构前备份。准备迁移至纯C环境与异步ROS2通信框架

File: src/my_bot/description/lidar.xacro (robot description, xacro)
@@ -3,13 +3,12 @@
     <!-- 激光雷达 link：安装在底盘上方的红色圆柱 -->
     <joint name="laser_joint" type="fixed">
-        <parent link="chassis" />
+        <parent link="base_link" />
         <child link="laser_frame" />
-        <!-- 根据你的底盘尺寸调整位置：X前方100mm，Z上方175mm -->
-        <origin xyz="0.1 0 0.175" rpy="0 0 0" />
+        <origin xyz="-0.025 0 0.1058" rpy="0 0 ${pi}" />
     </joint>
     <link name="laser_frame">
         <visual>
             <geometry>
-                <cylinder radius="0.05" length="0.04" />
+                <cylinder radius="0.025" length="0.02" />
             </geometry>
             <material name="red" />
@@ -17,8 +16,8 @@
         <collision>
             <geometry>
-                <cylinder radius="0.05" length="0.04" />
+                <cylinder radius="0.025" length="0.02" />
             </geometry>
         </collision>
-        <xacro:inertial_cylinder mass="0.1" length="0.04" radius="0.05">
+        <xacro:inertial_cylinder mass="0.01" length="0.025" radius="0.02">
             <origin xyz="0 0 0" rpy="0 0 0" />
         </xacro:inertial_cylinder>
@@ -42,6 +41,6 @@
                 </scan>
                 <range>
-                    <min>0.0699</min>
-                    <max>5.0001</max>
+                    <min>0.1</min>
+                    <max>5.0</max>
                 </range>
             </lidar>

File: src/my_bot/description/robot.urdf.xacro (robot description, xacro)
@@ -1,6 +1,6 @@
 <?xml version="1.0"?>
 <robot xmlns:xacro="http://www.ros.org/wiki/xacro" name="robot">
-    <xacro:arg name="sim_mode" default="true"/>
-    <xacro:arg name="ros2_control_config" default=""/>
+    <xacro:arg name="sim_mode" default="true" />
+    <xacro:arg name="ros2_control_config" default="" />
     <xacro:include filename="robot_core.xacro" />
     <!-- <xacro:include filename="gazebo_control.xacro"/> -->
@@ -12,3 +12,4 @@
     </xacro:unless>
     <xacro:include filename="lidar.xacro" />
+    <!-- <xacro:include filename="imu.xacro" /> -->
 </robot>

File: src/my_bot/description/robot_core.xacro (robot description, xacro)
@@ -1,4 +1,4 @@
 <?xml version="1.0"?>
-<robot xmlns:xacro="http://www.ros.org/wiki/xacro">
+<robot name="my_robot" xmlns:xacro="http://www.ros.org/wiki/xacro">
     <xacro:include filename="inertial_macros.xacro" />
     <!-- 颜色定义 -->
@@ -18,5 +18,22 @@
         <color rgba="1 0 0 1" />
     </material>
+    <!-- 车身结构 -->
     <link name="base_link">
+        <visual>
+            <origin xyz="-0.0275 0 0.0479" rpy="0 0 0" />
+            <geometry>
+                <box size="0.123 0.142 0.0958" />
+            </geometry>
+            <material name="white" />
+        </visual>
+        <collision>
+            <origin xyz="-0.0275 0 0.0479" rpy="0 0 0" />
+            <geometry>
+                <box size="0.123 0.142 0.0958" />
+            </geometry>
+        </collision>
+        <xacro:inertial_box mass="1.5" x="0.123" y="0.142" z="0.0958">
+            <origin xyz="-0.05 0 0.0479" rpy="0 0 0" />
+        </xacro:inertial_box>
     </link>
     <!-- BASE_FOOTPRINT -->
@@ -24,44 +41,20 @@
         <parent link="base_footprint" />
         <child link="base_link" />
-        <origin xyz="0 0 0.05" rpy="0 0 0" />
+        <!-- <origin xyz="0 0 0.05" rpy="0 0 0" /> -->
+        <origin xyz="0 0 0.012" rpy="0 0 0" />
     </joint>
     <link name="base_footprint">
     </link>
-    <!-- 车身结构 -->
-    <joint name="chassis_joint" type="fixed">
-        <parent link="base_link" />
-        <child link="chassis" />
-        <origin xyz="0 0 0" />
-    </joint>
-    <link name="chassis">
-        <visual>
-            <origin xyz="0.0 0 0.075" rpy="0 0 0" />
-            <geometry>
-                <box size="0.3 0.3 0.15" />
-            </geometry>
-            <material name="white" />
-        </visual>
-        <collision>
-            <origin xyz="0.0 0.0 0.075" rpy="0.0 0.0 0.0" />
-            <geometry>
-                <box size="0.3 0.3 0.15" />
-            </geometry>
-        </collision>
-        <xacro:inertial_box mass="3.5" x="0.3" y="0.3" z="0.15">
-            <origin xyz="0.0 0 0.075" rpy="0 0 0" />
-        </xacro:inertial_box>
-    </link>
+    <!-- 左轮 -->
     <joint name="left_wheel_joint" type="continuous">
         <parent link="base_link" />
         <child link="left_wheel" />
-        <origin xyz="0.0 0.175 0.0" rpy="-${pi/2} 0.0 0.0" />
+        <origin xyz="0.0 0.0658 0.0215" rpy="-${pi/2} 0.0 0.0" />
         <axis xyz="0.0 0.0 1.0" />
-        <limit effort="100.0" velocity="10.0" />
-        <dynamics damping="0.2" friction="0.2" />
     </joint>
     <link name="left_wheel">
         <visual>
             <geometry>
-                <cylinder radius="0.05" length="0.04" />
+                <cylinder radius="0.0335" length="0.031" />
             </geometry>
             <material name="blue" />
@@ -69,8 +62,8 @@
         <collision>
             <geometry>
-                <sphere radius="0.05" />
+                <cylinder radius="0.0335" length="0.031" />
             </geometry>
         </collision>
-        <xacro:inertial_cylinder mass="0.25" length="0.04" radius="0.05">
+        <xacro:inertial_cylinder mass="0.1" length="0.031" radius="0.0335">
             <origin xyz="0 0 0" rpy="0 0 0" />
         </xacro:inertial_cylinder>
@@ -78,39 +71,5 @@
     <gazebo reference="left_wheel">
         <mu1>1.0</mu1>
-        <mu2>0.5</mu2>
-        <kp>500000.0</kp>
-        <kd>10.0</kd>
-        <minDepth>0.001</minDepth>
-        <maxVel>0.1</maxVel>
-        <fdir1>1 0 0</fdir1>
-        <material>Gazebo/Blue</material>
-    </gazebo>
-    <joint name="right_wheel_joint" type="continuous">
-        <parent link="base_link" />
-        <child link="right_wheel" />
-        <origin xyz="0.0 -0.175 0.0" rpy="${pi/2} 0.0 0.0" />
-        <axis xyz="0.0 0.0 -1.0" />
-        <limit effort="100.0" velocity="10.0" />
-        <dynamics damping="0.2" friction="0.2" />
-    </joint>
-    <link name="right_wheel">
-        <visual>
-            <geometry>
-                <cylinder radius="0.05" length="0.04" />
-            </geometry>
-            <material name="blue" />
-        </visual>
-        <collision>
-            <geometry>
-                <sphere radius="0.05" />
-            </geometry>
-        </collision>
-        <xacro:inertial_cylinder mass="0.25" length="0.04" radius="0.05">
-            <origin xyz="0 0 0" rpy="0 0 0" />
-        </xacro:inertial_cylinder>
-    </link>
-    <gazebo reference="right_wheel">
-        <mu1>100000.0</mu1>
-        <mu2>100000.0</mu2>
+        <mu2>1.0</mu2>
         <kp>1000000.0</kp>
         <kd>100.0</kd>
@@ -120,14 +79,47 @@
         <material>Gazebo/Blue</material>
     </gazebo>
-    <!-- 前辅助轮 -->
-    <joint name="caster_front_joint" type="fixed">
-        <parent link="chassis" />
-        <child link="caster_front_wheel" />
-        <origin xyz="0.12 0 0" rpy="0 0 0" />
+    <!-- 右轮 -->
+    <joint name="right_wheel_joint" type="continuous">
+        <parent link="base_link" />
+        <child link="right_wheel" />
+        <origin xyz="0.0 -0.0658 0.0215" rpy="${pi/2} 0.0 0.0" />
+        <axis xyz="0.0 0.0 -1.0" />
     </joint>
-    <link name="caster_front_wheel">
+    <link name="right_wheel">
         <visual>
             <geometry>
-                <sphere radius="0.05" />
+                <cylinder radius="0.0335" length="0.031" />
+            </geometry>
+            <material name="blue" />
+        </visual>
+        <collision>
+            <geometry>
+                <cylinder radius="0.0335" length="0.031" />
+            </geometry>
+        </collision>
+        <xacro:inertial_cylinder mass="0.1" length="0.031" radius="0.0335">
+            <origin xyz="0 0 0" rpy="0 0 0" />
+        </xacro:inertial_cylinder>
+    </link>
+    <gazebo reference="right_wheel">
+        <mu1>1.0</mu1>
+        <mu2>1.0</mu2>
+        <kp>1000000.0</kp>
+        <kd>100.0</kd>
+        <minDepth>0.001</minDepth>
+        <maxVel>0.1</maxVel>
+        <fdir1>1 0 0</fdir1>
+        <material>Gazebo/Blue</material>
+    </gazebo>
+    <!-- 后辅助轮 -->
+    <joint name="caster_back_joint" type="fixed">
+        <parent link="base_link" />
+        <child link="caster_back_wheel" />
+        <origin xyz="-0.06445 0 0.008" rpy="0 0 0" />
+    </joint>
+    <link name="caster_back_wheel">
+        <visual>
+            <geometry>
+                <sphere radius="0.02" />
             </geometry>
             <material name="black" />
@@ -135,39 +127,8 @@
         <collision>
             <geometry>
-                <sphere radius="0.05" />
+                <sphere radius="0.02" />
             </geometry>
         </collision>
-        <xacro:inertial_sphere mass="0.1" radius="0.05">
-            <origin xyz="0 0 0" rpy="0 0 0" />
-        </xacro:inertial_sphere>
-    </link>
-    <gazebo reference="caster_front_wheel">
-        <mu1>0.0001</mu1>
-        <mu2>0.0001</mu2>
-        <kp>1000000.0</kp>
-        <kd>100.0</kd>
-        <minDepth>0.001</minDepth>
-        <maxVel>1.0</maxVel>
-        <material>Gazebo/Black</material>
-    </gazebo>
-    <!-- 后辅助轮 -->
-    <joint name="caster_back_joint" type="fixed">
-        <parent link="chassis" />
-        <child link="caster_back_wheel" />
-        <origin xyz="-0.12 0 0" rpy="0 0 0" />   <!-- 后方对称位置 -->
-    </joint>
-    <link name="caster_back_wheel">
-        <visual>
-            <geometry>
-                <sphere radius="0.05" />
-            </geometry>
-            <material name="black" />
-        </visual>
-        <collision>
-            <geometry>
-                <sphere radius="0.05" />
-            </geometry>
-        </collision>
-        <xacro:inertial_sphere mass="0.1" radius="0.05">
+        <xacro:inertial_sphere mass="0.1" radius="0.02">
             <origin xyz="0 0 0" rpy="0 0 0" />
         </xacro:inertial_sphere>

Commit message: Backup: 实机重构前备份。准备迁移至纯C环境与异步ROS2通信框架

File: src/my_bot/description/lidar.xacro (robot description, xacro)
@@ -3,13 +3,13 @@
     <!-- 激光雷达 link：安装在底盘上方的红色圆柱 -->
     <joint name="laser_joint" type="fixed">
-        <parent link="chassis" />
+        <parent link="base_link" />
         <child link="laser_frame" />
-        <!-- 根据你的底盘尺寸调整位置：X前方100mm，Z上方175mm -->
-        <origin xyz="0.1 0 0.175" rpy="0 0 0" />
+        <origin xyz="-0.025 0 0.1058" rpy="0 0 ${pi}" />
+        <!-- <origin xyz="-0.025 0 0.1158" rpy="0 0 0" /> -->
     </joint>
     <link name="laser_frame">
         <visual>
             <geometry>
-                <cylinder radius="0.05" length="0.04" />
+                <cylinder radius="0.025" length="0.02" />
             </geometry>
             <material name="red" />
@@ -17,8 +17,8 @@
         <collision>
             <geometry>
-                <cylinder radius="0.05" length="0.04" />
+                <cylinder radius="0.025" length="0.02" />
             </geometry>
         </collision>
-        <xacro:inertial_cylinder mass="0.1" length="0.04" radius="0.05">
+        <xacro:inertial_cylinder mass="0.01" length="0.025" radius="0.02">
             <origin xyz="0 0 0" rpy="0 0 0" />
         </xacro:inertial_cylinder>

File: src/my_bot/description/robot.urdf.xacro (robot description, xacro)
@@ -1,6 +1,6 @@
 <?xml version="1.0"?>
 <robot xmlns:xacro="http://www.ros.org/wiki/xacro" name="robot">
-    <xacro:arg name="sim_mode" default="true"/>
-    <xacro:arg name="ros2_control_config" default=""/>
+    <xacro:arg name="sim_mode" default="true" />
+    <xacro:arg name="ros2_control_config" default="" />
     <xacro:include filename="robot_core.xacro" />
     <!-- <xacro:include filename="gazebo_control.xacro"/> -->
@@ -12,3 +12,4 @@
     </xacro:unless>
     <xacro:include filename="lidar.xacro" />
+    <xacro:include filename="imu.xacro" />
 </robot>

Commit message: 仿真进入nav2，以与实机进行同步

File: src/my_bot/description/lidar.xacro (robot description, xacro)
@@ -35,5 +35,5 @@
                 <scan>
                     <horizontal>
-                        <samples>500</samples>
+                        <samples>720</samples>
                         <min_angle>-3.14159</min_angle>
                         <max_angle>3.14159</max_angle>
@@ -41,6 +41,6 @@
                 </scan>
                 <range>
-                    <min>0.1</min>
-                    <max>5.0</max>
+                    <min>0.05</min>
+                    <max>16.0</max>
                 </range>
             </lidar>

File: src/my_bot/description/robot.urdf.xacro (robot description, xacro)
@@ -4,6 +4,6 @@
     <xacro:arg name="ros2_control_config" default="" />
     <!-- LiDAR extrinsics (base_link -> laser_frame). Defaults match current model. -->
-    <xacro:arg name="lidar_x" default="-0.025" />
-    <xacro:arg name="lidar_y" default="0" />
+    <xacro:arg name="lidar_x" default="-0.026" />
+    <xacro:arg name="lidar_y" default="-0.0035" />
     <xacro:arg name="lidar_z" default="0.1058" />
     <xacro:arg name="lidar_roll" default="0" />

File: src/my_bot/description/robot_core.xacro (robot description, xacro)
@@ -23,5 +23,5 @@
             <origin xyz="-0.0275 0 0.0479" rpy="0 0 0" />
             <geometry>
-                <box size="0.123 0.142 0.0958" />
+                <box size="0.123 0.13 0.0958" />
             </geometry>
             <material name="white" />
@@ -30,8 +30,8 @@
             <origin xyz="-0.0275 0 0.0479" rpy="0 0 0" />
             <geometry>
-                <box size="0.123 0.142 0.0958" />
+                <box size="0.123 0.13 0.0958" />
             </geometry>
         </collision>
-        <xacro:inertial_box mass="1.5" x="0.123" y="0.142" z="0.0958">
+        <xacro:inertial_box mass="1.5" x="0.123" y="0.13" z="0.0958">
             <origin xyz="-0.05 0 0.0479" rpy="0 0 0" />
         </xacro:inertial_box>
@@ -50,5 +50,5 @@
         <parent link="base_link" />
         <child link="left_wheel" />
-        <origin xyz="0.0 0.0658 0.0215" rpy="-${pi/2} 0.0 0.0" />
+        <origin xyz="0.0 0.0875 0.023" rpy="-${pi/2} 0.0 0.0" />
         <axis xyz="0.0 0.0 1.0" />
     </joint>
@@ -56,5 +56,5 @@
         <visual>
             <geometry>
-                <cylinder radius="0.0335" length="0.031" />
+                <cylinder radius="0.035" length="0.027" />
             </geometry>
             <material name="blue" />
@@ -62,8 +62,8 @@
         <collision>
             <geometry>
-                <cylinder radius="0.0335" length="0.031" />
+                <cylinder radius="0.035" length="0.027" />
             </geometry>
         </collision>
-        <xacro:inertial_cylinder mass="0.1" length="0.031" radius="0.0335">
+        <xacro:inertial_cylinder mass="0.1" length="0.027" radius="0.035">
             <origin xyz="0 0 0" rpy="0 0 0" />
         </xacro:inertial_cylinder>
@@ -83,5 +83,5 @@
         <parent link="base_link" />
         <child link="right_wheel" />
-        <origin xyz="0.0 -0.0658 0.0215" rpy="${pi/2} 0.0 0.0" />
+        <origin xyz="0.0 -0.0875 0.023" rpy="${pi/2} 0.0 0.0" />
         <axis xyz="0.0 0.0 -1.0" />
     </joint>
@@ -89,5 +89,5 @@
         <visual>
             <geometry>
-                <cylinder radius="0.0335" length="0.031" />
+                <cylinder radius="0.035" length="0.027" />
             </geometry>
             <material name="blue" />
@@ -95,8 +95,8 @@
         <collision>
             <geometry>
-                <cylinder radius="0.0335" length="0.031" />
+                <cylinder radius="0.035" length="0.027" />
             </geometry>
         </collision>
-        <xacro:inertial_cylinder mass="0.1" length="0.031" radius="0.0335">
+        <xacro:inertial_cylinder mass="0.1" length="0.027" radius="0.035">
             <origin xyz="0 0 0" rpy="0 0 0" />
         </xacro:inertial_cylinder>

Commit message: MPPI调试阶段

File: src/my_bot/description/lidar.xacro (robot description, xacro)
@@ -5,5 +5,6 @@
         <parent link="base_link" />
         <child link="laser_frame" />
-        <origin xyz="$(arg lidar_x) $(arg lidar_y) $(arg lidar_z)" rpy="$(arg lidar_roll) $(arg lidar_pitch) $(arg lidar_yaw)" />
+        <origin xyz="$(arg lidar_x) $(arg lidar_y) $(arg lidar_z)"
+            rpy="$(arg lidar_roll) $(arg lidar_pitch) $(arg lidar_yaw)" />
     </joint>
     <link name="laser_frame">
@@ -41,6 +42,6 @@
                 </scan>
                 <range>
-                    <min>0.05</min>
-                    <max>16.0</max>
+                    <min>0.1</min>
+                    <max>4.0</max>
                 </range>
             </lidar>
