Commit message: feat(geometry): 实机几何同步 —— 双层 ⌀0.22 圆盘底盘
实机改用双层圆盘底盘，轮系与传感器安装位姿全变。按
docs/spec/2026-08-11-实机几何改动同步.md 同步仓库里的全部几何副本。

几何（相对 base_link；base_link = 第一层板下表面，离地 0.052）：
- 轮距 0.17152 → 0.192，轮半径 0.0334 → 0.035，轮厚 0.027 → 0.028
- 车身 box → cylinder(r=0.11, h=0.005) @(-0.047, 0)，新增 top_plate
- 脚轮 r 0.02 → 0.0125 @(-0.12, 0, -0.0395)
- 雷达 @(-0.047, 0, 0.072)，IMU @(0, -0.04, 0.032)
- 轮轴心与脚轮球心的 z 变为负值（底板抬高到 0.052 所致），不是笔误

控制器：
- hw/sim 两份 wheel_separation / wheel_radius 对齐实测值
- 三个 multiplier 复位 1.0（旧值是针对旧几何标的，已失效），待实机重标定

Nav2（6 份配置 x local+global = 12 处）：
- robot_radius 不可用：base_link 不在车体圆心上，圆心在其后方 0.047，
  取 robot_radius 须到 0.157，前方虚胖 94mm
- 改用 12 边形 footprint，按「圆盘 ∪ 两个驱动轮矩形」的支撑函数外切生成
- 轮子在 x=0 处突出盘缘 10.5mm，只按圆盘建会让轮子前外角露出 5.4/10.2mm

NeuPAN：length 0.18 → 0.22。DUNE 模型 diff_mybot.bin 仍按旧几何训成，
未重训，此期间实机导航只走 RPP。

其他：
- robot_core.xacro 挂 PosePublisher。Gazebo 默认不发 per-model pose 话题，
  此前 monitor.py 走备用分支的硬编码 index=9，在 home_4rooms.sdf 里读到的
  是 corridor_s_seg1（一堵墙），曾据此误判仿真打滑 61%
- 修正 my_bot/docs/README.md 不变量：几何真相源是 hw_controllers.yaml，
  不是固件 robot_config.h —— 那三个宏只服务于一个无调用点的 debug 函数

固件未改（依据同上，不参与运行链路）。

Co-Authored-By: Claude Opus 5 <noreply@anthropic.com>

File: src/my_bot/description/imu.xacro (robot description, xacro)
@@ -5,6 +5,6 @@
         <parent link="base_link"/>
         <child link="imu_link"/>
-        <!-- 车身几何中心 xy，中心 z -->
-        <origin xyz="-0.0275 0 0.0479" rpy="0 0 0"/>
+        <!-- 实测安装位：x=0，y 右偏 0.04，离地 0.084（base_link 上方 0.032）；朝向未变 -->
+        <origin xyz="0 -0.04 0.032" rpy="0 0 0"/>
     </joint>
     <link name="imu_link">

File: src/my_bot/description/robot.urdf.xacro (robot description, xacro)
@@ -4,7 +4,7 @@
     <xacro:arg name="ros2_control_config" default="" />
     <!-- LiDAR extrinsics (base_link -> laser_frame). Defaults match current model. -->
-    <xacro:arg name="lidar_x" default="-0.026" />
-    <xacro:arg name="lidar_y" default="-0.0035" />
-    <xacro:arg name="lidar_z" default="0.1058" />
+    <xacro:arg name="lidar_x" default="-0.047" />
+    <xacro:arg name="lidar_y" default="0" />
+    <xacro:arg name="lidar_z" default="0.072" />
     <xacro:arg name="lidar_roll" default="0" />
     <xacro:arg name="lidar_pitch" default="0" />

File: src/my_bot/description/robot_core.xacro (robot description, xacro)
@@ -18,29 +18,58 @@
         <color rgba="1 0 0 1" />
     </material>
-    <!-- 车身结构 -->
+    <!-- 车身结构：双层 ⌀0.22 圆盘（2026-08 底盘重做）
+         base_link = 第一层圆盘下表面所在平面，原点 = 两驱动轮轴心连线中点的投影。
+         圆盘圆心不在 base_link 上，而在其后方 0.047（差速车轮轴中点 ≠ 盘心）。 -->
     <link name="base_link">
         <visual>
-            <origin xyz="-0.0275 0 0.0479" rpy="0 0 0" />
-            <geometry>
-                <box size="0.123 0.13 0.0958" />
+            <origin xyz="-0.047 0 0.0025" rpy="0 0 0" />
+            <geometry>
+                <cylinder radius="0.11" length="0.005" />
             </geometry>
             <material name="white" />
         </visual>
         <collision>
-            <origin xyz="-0.0275 0 0.0479" rpy="0 0 0" />
-            <geometry>
-                <box size="0.123 0.13 0.0958" />
-            </geometry>
-        </collision>
-        <xacro:inertial_box mass="1.5" x="0.123" y="0.13" z="0.0958">
-            <origin xyz="-0.05 0 0.0479" rpy="0 0 0" />
-        </xacro:inertial_box>
-    </link>
+            <origin xyz="-0.047 0 0.0025" rpy="0 0 0" />
+            <geometry>
+                <cylinder radius="0.11" length="0.005" />
+            </geometry>
+        </collision>
+        <!-- 质量为估计值（整车实测质量待补），不影响 TF/里程计，只影响仿真动力学 -->
+        <xacro:inertial_cylinder mass="1.5" length="0.005" radius="0.11">
+            <origin xyz="-0.047 0 0.0025" rpy="0 0 0" />
+        </xacro:inertial_cylinder>
+    </link>
+    <!-- 第二层（顶板）：同规格 ⌀0.22 圆盘，由立柱撑开，顶面离地 0.16 -->
+    <joint name="top_plate_joint" type="fixed">
+        <parent link="base_link" />
+        <child link="top_plate" />
+        <origin xyz="-0.047 0 0.1055" rpy="0 0 0" />
+    </joint>
+    <link name="top_plate">
+        <visual>
+            <geometry>
+                <cylinder radius="0.11" length="0.005" />
+            </geometry>
+            <material name="white" />
+        </visual>
+        <collision>
+            <geometry>
+                <cylinder radius="0.11" length="0.005" />
+            </geometry>
+        </collision>
+        <!-- 质量为估计值，同上 -->
+        <xacro:inertial_cylinder mass="0.3" length="0.005" radius="0.11">
+            <origin xyz="0 0 0" rpy="0 0 0" />
+        </xacro:inertial_cylinder>
+    </link>
+    <gazebo reference="top_plate">
+        <material>Gazebo/White</material>
+    </gazebo>
     <!-- BASE_FOOTPRINT -->
     <joint name="base_footprint_joint" type="fixed">
         <parent link="base_footprint" />
         <child link="base_link" />
-        <!-- <origin xyz="0 0 0.05" rpy="0 0 0" /> -->
-        <origin xyz="0 0 0.012" rpy="0 0 0" />
+        <!-- 第一层圆盘下表面离地 0.052（实测） -->
+        <origin xyz="0 0 0.052" rpy="0 0 0" />
     </joint>
     <link name="base_footprint">
@@ -50,5 +79,6 @@
         <parent link="base_link" />
         <child link="left_wheel" />
-        <origin xyz="0.0 0.0875 0.023" rpy="-${pi/2} 0.0 0.0" />
+        <!-- z 为负：轮轴心在 base_link（板下表面, 离地 0.052）下方 0.017，即离地 0.035 = 轮半径 -->
+        <origin xyz="0.0 0.096 -0.017" rpy="-${pi/2} 0.0 0.0" />
         <axis xyz="0.0 0.0 1.0" />
     </joint>
@@ -56,5 +86,5 @@
         <visual>
             <geometry>
-                <cylinder radius="0.035" length="0.027" />
+                <cylinder radius="0.035" length="0.028" />
             </geometry>
             <material name="blue" />
@@ -62,8 +92,8 @@
         <collision>
             <geometry>
-                <cylinder radius="0.035" length="0.027" />
-            </geometry>
-        </collision>
-        <xacro:inertial_cylinder mass="0.1" length="0.027" radius="0.035">
+                <cylinder radius="0.035" length="0.028" />
+            </geometry>
+        </collision>
+        <xacro:inertial_cylinder mass="0.1" length="0.028" radius="0.035">
             <origin xyz="0 0 0" rpy="0 0 0" />
         </xacro:inertial_cylinder>
@@ -83,5 +113,6 @@
         <parent link="base_link" />
         <child link="right_wheel" />
-        <origin xyz="0.0 -0.0875 0.023" rpy="${pi/2} 0.0 0.0" />
+        <!-- z 为负，同左轮 -->
+        <origin xyz="0.0 -0.096 -0.017" rpy="${pi/2} 0.0 0.0" />
         <axis xyz="0.0 0.0 -1.0" />
     </joint>
@@ -89,5 +120,5 @@
         <visual>
             <geometry>
-                <cylinder radius="0.035" length="0.027" />
+                <cylinder radius="0.035" length="0.028" />
             </geometry>
             <material name="blue" />
@@ -95,8 +126,8 @@
         <collision>
             <geometry>
-                <cylinder radius="0.035" length="0.027" />
-            </geometry>
-        </collision>
-        <xacro:inertial_cylinder mass="0.1" length="0.027" radius="0.035">
+                <cylinder radius="0.035" length="0.028" />
+            </geometry>
+        </collision>
+        <xacro:inertial_cylinder mass="0.1" length="0.028" radius="0.035">
             <origin xyz="0 0 0" rpy="0 0 0" />
         </xacro:inertial_cylinder>
@@ -116,10 +147,11 @@
         <parent link="base_link" />
         <child link="caster_back_wheel" />
-        <origin xyz="-0.06445 0 0.008" rpy="0 0 0" />
+        <!-- WHEELTEC 万向轮 Ø25，球心在轮轴中点后方 0.12；z 为负，球心离地 0.0125 = 球半径 -->
+        <origin xyz="-0.12 0 -0.0395" rpy="0 0 0" />
     </joint>
     <link name="caster_back_wheel">
         <visual>
             <geometry>
-                <sphere radius="0.02" />
+                <sphere radius="0.0125" />
             </geometry>
             <material name="black" />
@@ -127,8 +159,8 @@
         <collision>
             <geometry>
-                <sphere radius="0.02" />
-            </geometry>
-        </collision>
-        <xacro:inertial_sphere mass="0.1" radius="0.02">
+                <sphere radius="0.0125" />
+            </geometry>
+        </collision>
+        <xacro:inertial_sphere mass="0.05" radius="0.0125">
             <origin xyz="0 0 0" rpy="0 0 0" />
         </xacro:inertial_sphere>
@@ -143,3 +175,31 @@
         <material>Gazebo/Black</material>
     </gazebo>
+    <!-- ═══ Gazebo 地面真值发布器 ═══════════════════════════════════════════
+         把模型位姿发到 gz 话题 /model/my_bot/pose，再由 config/gz_bridge.yaml
+         桥接成 ROS 的 /gz/model/my_bot/pose（PoseStamped）。
+         为什么必须有它（2026-08-12 加）：
+         Gazebo 默认【不】发布 per-model 的 pose 话题，只发世界级的
+         /world/default/pose/info（Pose_V，含所有 model+link+visual）。
+         而 Pose_V 桥接成 geometry_msgs/PoseArray 后【丢失 name 字段】，
+         下游只能靠数组下标定位机器人 —— 下标随世界里模型的数量和顺序变，必然过期。
+         实测教训：python/monitor.py 与 gz_pose_monitor.py 的备用分支都硬编码
+         WORLD_POSES_INDEX = 9，而在 worlds/home_4rooms.sdf 里 index=9 是
+         corridor_s_seg1（一堵墙），my_bot 实际在 index=38。也就是说在挂上本插件之前，
+         这两个脚本显示的「Gazebo 真值」读的根本不是机器人。
+         两个脚本都已写好「优先用单话题、其次用 PoseArray」的逻辑，所以本插件一生效
+         它们就自动走对通道，无需改动脚本。
+         注：本标签在实机（sim_mode:=false）下会被 robot_state_publisher 忽略，无副作用。
+    ═══════════════════════════════════════════════════════════════════════ -->
+    <gazebo>
+        <plugin filename="gz-sim-pose-publisher-system"
+                name="gz::sim::systems::PosePublisher">
+            <publish_model_pose>true</publish_model_pose>
+            <publish_link_pose>false</publish_link_pose>
+            <publish_collision_pose>false</publish_collision_pose>
+            <publish_visual_pose>false</publish_visual_pose>
+            <publish_nested_model_pose>false</publish_nested_model_pose>
+            <use_pose_vector_msg>false</use_pose_vector_msg>
+            <update_frequency>50</update_frequency>
+        </plugin>
+    </gazebo>
 </robot>
